File: spacex-sbc.kicad_pcb (KiCad board)
At the start: 2 copper layers, 2 parts, among them J1 Conn_02x13_Odd_Even, U1 STM32MP157AAAx

Commit message: saved
Parts:
- removed the U1 at (182.7, 84.5)
- added U1: STM32MP135AAFx, Package_BGA:ST_TFBGA-320_11x11mm_Layout21x21_P0.5mm, F.Cu at (183.9, 78.1)
- added U1: STM32MP135AAFx, Package_BGA:ST_TFBGA-320_11x11mm_Layout21x21_P0.5mm, F.Cu at (183.6, 91.9)
- added U1: STM32MP135AAFx, Package_BGA:ST_TFBGA-320_11x11mm_Layout21x21_P0.5mm, F.Cu at (170.5, 78.2)
- added U1: STM32MP135AAFx, Package_BGA:ST_TFBGA-320_11x11mm_Layout21x21_P0.5mm, F.Cu at (170.6, 91.8)
- added U2: ATSAMA5D21, Package_BGA:ST_LFBGA-354_16x16mm_Layout19x19_P0.8mm, F.Cu at (154.5, 86.2)
Routing:
- net unconnected-(U2B-PB3-PadB5): track 0.00 -> 2.06 mm
- net unconnected-(U2F-DDR_D3-PadB9): track 0.00 -> 2.04 mm
- net unconnected-(U2F-DDR_DQS0-PadB8): track 0.00 -> 2.00 mm
- net unconnected-(U2B-PB2-PadB6): track 0.00 -> 1.97 mm
- net unconnected-(U2F-DDR_D0-PadB7): track 0.00 -> 1.95 mm
- net unconnected-(U2F-DDR_D4-PadA9): track 0.00 -> 1.93 mm
- net unconnected-(U2F-DDR_D6-PadA10): track 0.00 -> 1.88 mm
- net unconnected-(U2B-PB1-PadA5): track 0.00 -> 1.80 mm
- net unconnected-(U1-PC11-PadB18): track 0.00 -> 1.72 mm
- net unconnected-(U2F-DDR_DQSN0-PadA8): track 0.00 -> 1.64 mm
- net unconnected-(U2F-DDR_D1-PadA7): track 0.00 -> 1.61 mm
- net unconnected-(U2B-PB0-PadA6): track 0.00 -> 1.43 mm
- net unconnected-(U1-PF0-PadA16): track 0.00 -> 0.58 mm, vias 0 -> 1

Commit message: mostly mocked up
Parts:
- removed the U1 at (183.9, 78.1)
- removed the U1 at (183.6, 91.9)
- removed the U1 at (170.5, 78.2)
- removed the U1 at (170.6, 91.8)
- added C1: C, Capacitor_SMD:C_1210_3225Metric, F.Cu at (140.7, 85.7)
- added C10: C_Polarized, Capacitor_SMD:CP_Elec_5x3, F.Cu at (191.8, 98.9)
- added C11: C, Capacitor_SMD:C_1206_3216Metric, F.Cu at (204.4, 108.8)
- added C12: C, Capacitor_SMD:C_1206_3216Metric, F.Cu at (206.7, 108.8)
- added C13: C, Capacitor_SMD:C_0402_1005Metric, F.Cu at (196.8, 104.9)
- added C14: 12pF, Capacitor_SMD:C_0402_1005Metric, F.Cu at (130.2, 126.9)
- added C15: 12pF, Capacitor_SMD:C_0402_1005Metric, F.Cu at (133.2, 126.9)
- added C16: C_Polarized, Capacitor_SMD:CP_Elec_5x3, F.Cu at (191.8, 114.3)
- added C2: C, Capacitor_SMD:C_1206_3216Metric, F.Cu at (145.2, 85.6)
- added C3: C, Capacitor_SMD:C_0805_2012Metric, F.Cu at (149.4, 85.7)
- added C4: C, Capacitor_SMD:C_0603_1608Metric, F.Cu at (152.9, 85.7)
- added C5: C, Capacitor_SMD:C_0402_1005Metric, F.Cu at (155.9, 85.7)
- added C6: C, Capacitor_SMD:C_0201_0603Metric, F.Cu at (158.7, 85.6)
- added C7: C, Capacitor_SMD:C_1206_3216Metric, F.Cu at (204.4, 93.4)
- added C8: C, Capacitor_SMD:C_1206_3216Metric, F.Cu at (206.7, 93.4)
- added C9: C, Capacitor_SMD:C_0402_1005Metric, F.Cu at (196.8, 89.5)
- added D1: D_Schottky, Diode_SMD:D_0603_1608Metric, F.Cu at (201.3, 89.7)
- added D2: D_Schottky, Diode_SMD:D_0603_1608Metric, F.Cu at (201.3, 105.1)
- added J2: MX34 40-PIN, Connector_JAE:JAE_LY20-40P-DLT1_2x20_P2.00mm_Horizontal, F.Cu at (81.9, 70.6)
- added J3: Conn_01x02, Connector_Molex:Molex_Micro-Fit_3.0_43650-0200_1x02_P3.00mm_Horizontal, F.Cu at (215.6, 108.4)
- added L1: L_Iron, Inductor_SMD:L_6.3x6.3_H3, F.Cu at (189.7, 92.2)
- added L2: L_Iron, Inductor_SMD:L_6.3x6.3_H3, F.Cu at (189.7, 107.6)
- added R1: R_US, Resistor_SMD:R_0402_1005Metric, F.Cu at (195.9, 96.6)
- added R2: R_US, Resistor_SMD:R_0402_1005Metric, F.Cu at (197.9, 96.6)
- added R3: R_US, Resistor_SMD:R_0402_1005Metric, F.Cu at (195.9, 112.0)
- added R4: R_US, Resistor_SMD:R_0402_1005Metric, F.Cu at (197.9, 112.0)
- added R5: R_US, Resistor_SMD:R_0402_1005Metric, F.Cu at (167.0, 107.8)
- added R6: R_US, Resistor_SMD:R_0402_1005Metric, F.Cu at (197.5, 49.6)
- added U1: STM32MP135AAFx, Package_BGA:ST_TFBGA-320_11x11mm_Layout21x21_P0.5mm, F.Cu at (133.7, 98.1)
- added U10: MCP16501TE-E/RMB, Package_DFN_QFN:QFN-24-1EP_4x4mm_P0.5mm_EP2.7x2.7mm, F.Cu at (218.6, 94.6)
- added U3: ATSAMA5D21, Package_BGA:Microchip_TFBGA-196_11x11mm_Layout14x14_P0.75mm_SMD, F.Cu at (167.3, 99.1)
- added U4: MAX3221, Package_SO:SSOP-16_4.4x5.2mm_P0.65mm, F.Cu at (161.0, 64.1)
- added U5: MT41K256M16TW, Package_BGA:Micron_FBGA-96_8x14mm_Layout9x16_P0.8mm, F.Cu at (193.6, 58.2)
- added U6: TPS5430DDA, Package_SO:TI_SO-PowerPAD-8_ThermalVias, F.Cu at (199.5, 93.3)
- added U7: MCP2562-E-SN, Package_SO:SOIC-8_3.9x4.9mm_P1.27mm, F.Cu at (138.7, 64.8)
- added U8: 28F400, Package_BGA:BGA-63_9x11mm_Layout10x12_P0.8mm, F.Cu at (193.7, 74.8)
- added U9: TPS5430DDA, Package_SO:TI_SO-PowerPAD-8_ThermalVias, F.Cu at (199.5, 108.7)
- added Y1: 8MHz, Crystal:Crystal_SMD_1210-4Pin_1.2x1.0mm, F.Cu at (131.7, 126.9)
- J1: value Conn_02x13_Odd_Even -> 26PIN_RPI_HEADER
- U2: value ATSAMA5D21 -> STM32MP131AAEx; footprint Package_BGA:ST_LFBGA-354_16x16mm_Layout19x19_P0.8mm -> Package_BGA:LFBGA-289_14x14mm_Layout17x17_P0.8mm
- moved J1 65.7 mm to (181.2, 128.0), turned to 90 degrees
- moved U2 13.3 mm to (150.2, 98.8)
Connections:
- J1 pad 1: unconnected-(J1-Pin_1-Pad1) -> Net-(J1-Pin_1)
- J1 pad 10: unconnected-(J1-Pin_10-Pad10) -> RPI_GPIO15
- J1 pad 11: unconnected-(J1-Pin_11-Pad11) -> RPI_GPIO17
- J1 pad 12: unconnected-(J1-Pin_12-Pad12) -> RPI_GPIO18
- J1 pad 13: unconnected-(J1-Pin_13-Pad13) -> RPI_GPIO27
- J1 pad 14: unconnected-(J1-Pin_14-Pad14) -> GND
- J1 pad 15: unconnected-(J1-Pin_15-Pad15) -> RPI_GPIO22
- J1 pad 16: unconnected-(J1-Pin_16-Pad16) -> RPI_GPIO23
- J1 pad 17: unconnected-(J1-Pin_17-Pad17) -> Net-(J1-Pin_1)
- J1 pad 18: unconnected-(J1-Pin_18-Pad18) -> RPI_GPIO24
- J1 pad 19: unconnected-(J1-Pin_19-Pad19) -> RPI_GPIO10
- J1 pad 2: unconnected-(J1-Pin_2-Pad2) -> +5V
- J1 pad 20: unconnected-(J1-Pin_20-Pad20) -> GND
- J1 pad 21: unconnected-(J1-Pin_21-Pad21) -> RPI_GPIO9
- J1 pad 22: unconnected-(J1-Pin_22-Pad22) -> RPI_GPIO25
- J1 pad 23: unconnected-(J1-Pin_23-Pad23) -> RPI_GPIO11
- J1 pad 24: unconnected-(J1-Pin_24-Pad24) -> RPI_GPIO8
- J1 pad 25: unconnected-(J1-Pin_25-Pad25) -> GND
- J1 pad 26: unconnected-(J1-Pin_26-Pad26) -> RPI_GPIO7
- J1 pad 3: unconnected-(J1-Pin_3-Pad3) -> RPI_GPIO2
- J1 pad 4: unconnected-(J1-Pin_4-Pad4) -> +5V
- J1 pad 5: unconnected-(J1-Pin_5-Pad5) -> RPI_GPIO3
- J1 pad 6: unconnected-(J1-Pin_6-Pad6) -> GND
- J1 pad 7: unconnected-(J1-Pin_7-Pad7) -> RPI_GPIO4
- J1 pad 8: unconnected-(J1-Pin_8-Pad8) -> RPI_GPIO14
- J1 pad 9: unconnected-(J1-Pin_9-Pad9) -> GND
- U2 pad A1: unconnected-(U2B-PB10-PadA1) -> Net-(U2-VSS-PadA1)
- U2 pad A15: (no net) -> unconnected-(U2-PD2-PadA15)
- U2 pad A16: (no net) -> unconnected-(U2-PC9-PadA16)
- U2 pad A17: (no net) -> Net-(U2-VSS-PadA1)
- U2 pad B15: (no net) -> unconnected-(U2-PC12-PadB15)
- U2 pad B16: (no net) -> unconnected-(U2-DDR_DQ4-PadB16)
- U2 pad B17: (no net) -> unconnected-(U2-DDR_DQ0-PadB17)
- U2 pad C12: Net-(U2F-DDR_VREF-PadC12) -> unconnected-(U2-VDDSD1-PadC12)
- U2 pad C15: (no net) -> unconnected-(U2-DDR_DQ1-PadC15)
- U2 pad C16: (no net) -> unconnected-(U2-DDR_DQS0N-PadC16)
- U2 pad C17: (no net) -> unconnected-(U2-DDR_DQS0P-PadC17)
- U2 pad C6: Net-(U2F-VDDIODDR-PadC6) -> unconnected-(U2-PD12-PadC6)
- U2 pad C7: Net-(U2F-GNDIODDR-PadC7) -> unconnected-(U2-PD15-PadC7)
- U2 pad C8: unconnected-(U2F-DDR_D2-PadC8) -> Net-(U2-VSS-PadA1)
- U2 pad D12: Net-(U2F-GNDIODDR-PadC7) -> Net-(U2-VSS-PadA1)
- U2 pad D15: (no net) -> unconnected-(U2-DDR_DQM0-PadD15)
- U2 pad D16: (no net) -> unconnected-(U2-DDR_DQ5-PadD16)
- U2 pad D17: (no net) -> unconnected-(U2-DDR_DQ3-PadD17)
- U2 pad D3: unconnected-(U2B-PB24-PadD3) -> Net-(U2-VSS-PadA1)
- U2 pad D7: Net-(U2E-VDDIOP0-PadD7) -> unconnected-(U2-PG0-PadD7)
- U2 pad E10: Net-(U2F-VDDIODDR-PadC6) -> unconnected-(U2-PB13-PadE10)
- U2 pad E12: Net-(U2F-VDDIODDR-PadC6) -> Net-(U2-VDDQ_DDR-PadE12)
- U2 pad E15: (no net) -> unconnected-(U2-DDR_DQ7-PadE15)
- U2 pad E16: (no net) -> unconnected-(U2-DDR_A5-PadE16)
- U2 pad E17: (no net) -> unconnected-(U2-DDR_RESETN-PadE17)
- U2 pad E4: Net-(U2E-GNDIOP0-PadE4) -> unconnected-(U2-PD0-PadE4)
- U2 pad E5: unconnected-(U2B-PB15-PadE5) -> Net-(U2-VSS-PadA1)
- U2 pad E7: Net-(U2E-GNDIOP0-PadE4) -> unconnected-(U2-PD4-PadE7)
- U2 pad E8: Net-(U2E-VDDCORE-PadE8) -> unconnected-(U2-PD9-PadE8)
- U2 pad E9: Net-(U2F-GNDIODDR-PadC7) -> unconnected-(U2-PF2-PadE9)
- U2 pad F10: unconnected-(U2F-DDR_CAL-PadF10) -> Net-(U2-VDD-PadF10)
- U2 pad F11: unconnected-(U2F-DDR_CS-PadF11) -> Net-(U2-VDD-PadF10)
- U2 pad F12: Net-(U2F-GNDIODDR-PadC7) -> Net-(U2-VDDQ_DDR-PadE12)
- U2 pad F13: unconnected-(U2F-DDR_BA0-PadF13) -> Net-(U2-VSS-PadA1)
- U2 pad F15: (no net) -> Net-(U2-VSS-PadA1)
- U2 pad F17: (no net) -> unconnected-(U2-DDR_A2-PadF17)
- U2 pad F4: Net-(U2E-VDDIOP0-PadD7) -> unconnected-(U2-PH2-PadF4)
- U2 pad F6: unconnected-(U2B-PB29-PadF6) -> Net-(U2-VDDCPU-PadF6)
- U2 pad F7: unconnected-(U2B-PB31-PadF7) -> Net-(U2-VDD-PadF10)
- U2 pad F8: Net-(U2E-GNDCORE-PadF8) -> Net-(U2-VDDCPU-PadF6)
- U2 pad F9: unconnected-(U2F-DDR_A10-PadF9) -> Net-(U2-VDDCPU-PadF6)
- U2 pad G10: Net-(U2F-VDDIODDR-PadC6) -> Net-(U2-VSS-PadA1)
- U2 pad G11: Net-(U2F-GNDIODDR-PadC7) -> Net-(U2-VSS-PadA1)
- U2 pad G12: Net-(U2F-VDDIODDR-PadC6) -> Net-(U2-VDDQ_DDR-PadE12)
- U2 pad G15: (no net) -> unconnected-(U2-DDR_A3-PadG15)
- U2 pad G16: (no net) -> unconnected-(U2-DDR_A0-PadG16)
- U2 pad G17: (no net) -> unconnected-(U2-DDR_BA0-PadG17)
- U2 pad G6: unconnected-(U2D-PD14-PadG6) -> Net-(U2-VDD-PadF10)
- U2 pad G7: Net-(U2E-GNDCORE-PadF8) -> Net-(U2-VSS-PadA1)
- U2 pad G8: Net-(U2E-VDDCORE-PadE8) -> Net-(U2-VSS-PadA1)
- U2 pad G9: Net-(U2E-GNDCORE-PadF8) -> Net-(U2-VSS-PadA1)
- U2 pad H10: Net-(U2F-GNDIODDR-PadC7) -> Net-(U2-VDDCORE-PadH10)
- U2 pad H11: Net-(U2F-VDDIODDR-PadC6) -> Net-(U2-VSS-PadA1)
- U2 pad H12: Net-(U2F-DDR_VREF-PadC12) -> Net-(U2-VDDQ_DDR-PadE12)
- U2 pad H14: unconnected-(U2F-DDR_D9-PadH14) -> Net-(U2-VSS-PadA1)
- U2 pad H15: (no net) -> unconnected-(U2-DDR_ODT-PadH15)
- U2 pad H17: (no net) -> unconnected-(U2-DDR_RASN-PadH17)
- U2 pad H2: Net-(U2E-VDDANA-PadH2) -> unconnected-(U2-PI3-PadH2)
- U2 pad H6: unconnected-(U2D-PD12-PadH6) -> Net-(U2-VDDCPU-PadF6)
- U2 pad H7: Net-(U2E-GNDCORE-PadF8) -> Net-(U2-VSS-PadA1)
- U2 pad H8: Net-(U2E-VDDCORE-PadE8) -> Net-(U2-VDDCORE-PadH10)
- U2 pad H9: Net-(U2E-VDDCORE-PadE8) -> Net-(U2-VDDCORE-PadH10)
- U2 pad J10: Net-(U2F-VDDIODDR-PadC6) -> Net-(U2-VDDCORE-PadH10)
- U2 pad J11: Net-(U2F-GNDIODDR-PadC7) -> Net-(U2-VSS-PadA1)
- U2 pad J12: unconnected-(U2F-DDR_D14-PadJ12) -> Net-(U2-VDDQ_DDR-PadE12)
- U2 pad J13: unconnected-(U2F-DDR_D10-PadJ13) -> Net-(U2-VDDCORE-PadH10)
- U2 pad J15: (no net) -> unconnected-(U2-DDR_CASN-PadJ15)
- U2 pad J16: (no net) -> unconnected-(U2-DDR_CLKP-PadJ16)
- U2 pad J17: (no net) -> unconnected-(U2-DDR_CLKN-PadJ17)
- U2 pad J2: Net-(U2E-GNDANA-PadJ2) -> unconnected-(U2-VBAT-PadJ2)
- U2 pad J4: Net-(U2E-GNDCORE-PadF8) -> unconnected-(U2-VSS_PLL-PadJ4)
- U2 pad J5: Net-(U2E-VDDCORE-PadE8) -> unconnected-(U2-VDD_PLL-PadJ5)
- U2 pad J6: unconnected-(U2I-GNDAUDIOPLL-PadJ6) -> Net-(U2-VDDCPU-PadF6)
- U2 pad J7: unconnected-(U2I-CLK_AUDIO-PadJ7) -> Net-(U2-VSS-PadA1)
- U2 pad J8: unconnected-(U2C-PC5-PadJ8) -> Net-(U2-VDDCORE-PadH10)
- U2 pad J9: unconnected-(U2C-PC8-PadJ9) -> Net-(U2-VSS-PadA1)
- U2 pad K10: unconnected-(U2C-PC3-PadK10) -> Net-(U2-VDDCORE-PadH10)
- U2 pad K11: unconnected-(U2G-VDDFUSE-PadK11) -> Net-(U2-VSS-PadA1)
- U2 pad K12: unconnected-(U2F-DDR_D15-PadK12) -> Net-(U2-VDDQ_DDR-PadE12)
- U2 pad K15: (no net) -> unconnected-(U2-DDR_A1-PadK15)
- U2 pad K17: (no net) -> unconnected-(U2-DDR_A12-PadK17)
- U2 pad K3: Net-(U2E-VDDANA-PadH2) -> Net-(U2-VSS-PadA1)
- U2 pad K4: Net-(U2E-GNDANA-PadJ2) -> unconnected-(U2-PC13-PadK4)
- U2 pad K6: unconnected-(U2I-VDDAUDIOPLL-PadK6) -> Net-(U2-VDD-PadF10)
- U2 pad K7: unconnected-(U2G-VDDUTMII-PadK7) -> Net-(U2-VSS-PadA1)
- U2 pad K8: Net-(U2E-VDDIOP1-PadK8) -> Net-(U2-VDDCORE-PadH10)
- U2 pad K9: Net-(U2E-GNDIOP1-PadK9) -> Net-(U2-VDDCORE-PadH10)
- U2 pad L10: unconnected-(U2A-PA25-PadL10) -> Net-(U2-VSS-PadA1)
- U2 pad L11: Net-(U2E-VDDIOP1-PadK8) -> Net-(U2-VSS-PadA1)
- U2 pad L12: Net-(U2E-GNDIOP1-PadK9) -> Net-(U2-VDDQ_DDR-PadE12)
- U2 pad L15: (no net) -> unconnected-(U2-DDR_A8-PadL15)
- U2 pad L16: (no net) -> unconnected-(U2-DDR_BA1-PadL16)
- U2 pad L17: (no net) -> unconnected-(U2-DDR_A14-PadL17)
- U2 pad L6: unconnected-(U2E-GNDDPLL-PadL6) -> Net-(U2-VDD-PadF10)
- U2 pad L7: unconnected-(U2G-VBG-PadL7) -> Net-(U2-VSS-PadA1)
- U2 pad L8: unconnected-(U2G-GNDUTMII-PadL8) -> Net-(U2-VSS-PadA1)
- U2 pad L9: unconnected-(U2A-PA18-PadL9) -> Net-(U2-VSS-PadA1)
- U2 pad M10: unconnected-(U2A-PA21-PadM10) -> Net-(U2-VDD-PadF10)
- U2 pad M11: unconnected-(U2A-PA28-PadM11) -> Net-(U2-VDD-PadF10)
- U2 pad M12: unconnected-(U2A-PA31-PadM12) -> Net-(U2-VDDQ_DDR-PadE12)
- U2 pad M15: (no net) -> Net-(U2-VSS-PadA1)
- U2 pad M17: (no net) -> unconnected-(U2-DDR_A6-PadM17)
- U2 pad M6: unconnected-(U2H-PIOBU5-PadM6) -> Net-(U2-VDD-PadF10)
- U2 pad M7: unconnected-(U2G-VDDUTMIC-PadM7) -> Net-(U2-VDD-PadF10)
- U2 pad M8: unconnected-(U2G-GNDUTMIC-PadM8) -> Net-(U2-VDD-PadF10)
- U2 pad M9: unconnected-(U2A-PA20-PadM9) -> Net-(U2-VDD-PadF10)
- U2 pad N12: unconnected-(U2A-PA30-PadN12) -> Net-(U2-VDDQ_DDR-PadE12)
- U2 pad N15: (no net) -> unconnected-(U2-DDR_DQ10-PadN15)
- U2 pad N16: (no net) -> unconnected-(U2-DDR_DQ8-PadN16)
- U2 pad N17: (no net) -> unconnected-(U2-DDR_ZQ-PadN17)
- U2 pad N4: unconnected-(U2H-PIOBU3-PadN4) -> Net-(U2-VSS-PadA1)
- U2 pad P11: unconnected-(U2A-PA26-PadP11) -> Net-(U2-VSS-PadA1)
- U2 pad P15: (no net) -> unconnected-(U2-DDR_DQ11-PadP15)
- U2 pad P17: (no net) -> unconnected-(U2-DDR_DQ9-PadP17)
- U2 pad R1: (no net) -> unconnected-(U2-PG2-PadR1)
- U2 pad R10: (no net) -> unconnected-(U2-PF15-PadR10)
- U2 pad R11: (no net) -> unconnected-(U2-VDDA1V8_REG-PadR11)
- U2 pad R12: (no net) -> unconnected-(U2-PI6-PadR12)
- U2 pad R13: (no net) -> unconnected-(U2-VDD_PLL2-PadR13)
- U2 pad R14: (no net) -> unconnected-(U2-PH5-PadR14)
- U2 pad R15: (no net) -> unconnected-(U2-DDR_DQ12-PadR15)
- U2 pad R16: (no net) -> unconnected-(U2-DDR_DQS1N-PadR16)
- U2 pad R17: (no net) -> unconnected-(U2-DDR_DQS1P-PadR17)
- U2 pad R2: (no net) -> unconnected-(U2-PH3-PadR2)
- U2 pad R3: (no net) -> unconnected-(U2-PWR_CPU_ON-PadR3)
- U2 pad R4: (no net) -> unconnected-(U2-PA1-PadR4)
- U2 pad R5: (no net) -> Net-(U2-VSS-PadA1)
- U2 pad R6: (no net) -> unconnected-(U2-VREF+-PadR6)
- U2 pad R7: (no net) -> unconnected-(U2-PC5-PadR7)
- U2 pad R8: (no net) -> Net-(U2-VSS-PadA1)
- U2 pad R9: (no net) -> Net-(U2-VDD-PadF10)
- U2 pad T1: (no net) -> unconnected-(U2-PG12-PadT1)
- U2 pad T10: (no net) -> unconnected-(U2-PDR_ON-PadT10)
- U2 pad T11: (no net) -> unconnected-(U2-USB_DP2-PadT11)
- U2 pad T12: (no net) -> unconnected-(U2-PA14-PadT12)
- U2 pad T13: (no net) -> unconnected-(U2-USB_DP1-PadT13)
- U2 pad T14: (no net) -> unconnected-(U2-BYPASS_REG1V8-PadT14)
- U2 pad T15: (no net) -> unconnected-(U2-PH4-PadT15)
- U2 pad T16: (no net) -> unconnected-(U2-DDR_DQ15-PadT16)
- U2 pad T17: (no net) -> unconnected-(U2-DDR_DQ14-PadT17)
- U2 pad T2: (no net) -> unconnected-(U2-PA11-PadT2)
- U2 pad T3: (no net) -> unconnected-(U2-PC0-PadT3)
- U2 pad T4: (no net) -> unconnected-(U2-PF12-PadT4)
- U2 pad T5: (no net) -> unconnected-(U2-PC3-PadT5)
- U2 pad T6: (no net) -> unconnected-(U2-PF11-PadT6)
- U2 pad T7: (no net) -> unconnected-(U2-PB1-PadT7)
- U2 pad T8: (no net) -> unconnected-(U2-PA6-PadT8)
- U2 pad T9: (no net) -> unconnected-(U2-PE5-PadT9)
- U2 pad U1: (no net) -> Net-(U2-VSS-PadA1)
- U2 pad U10: (no net) -> unconnected-(U2-NRST-PadU10)
- U2 pad U11: (no net) -> unconnected-(U2-USB_DM2-PadU11)
- U2 pad U12: (no net) -> unconnected-(U2-USB_RREF-PadU12)
- U2 pad U13: (no net) -> unconnected-(U2-USB_DM1-PadU13)
- U2 pad U14: (no net) -> unconnected-(U2-PI4-PadU14)
- U2 pad U15: (no net) -> unconnected-(U2-PA10-PadU15)
- U2 pad U16: (no net) -> unconnected-(U2-PI7-PadU16)
- U2 pad U17: (no net) -> Net-(U2-VSS-PadA1)
- U2 pad U2: (no net) -> unconnected-(U2-PA7-PadU2)
- U2 pad U3: (no net) -> unconnected-(U2-PA0-PadU3)
- U2 pad U4: (no net) -> unconnected-(U2-PA5-PadU4)
- U2 pad U5: (no net) -> unconnected-(U2-PA4-PadU5)
- U2 pad U6: (no net) -> unconnected-(U2-PC4-PadU6)
- U2 pad U7: (no net) -> unconnected-(U2-PB0-PadU7)
- U2 pad U8: (no net) -> unconnected-(U2-PC1-PadU8)
- U2 pad U9: (no net) -> unconnected-(U2-PC2-PadU9)
Routing:
- net unconnected-(U2-PE1-PadB5): track 2.06 -> 0.00 mm
- net unconnected-(U2-PF1-PadB9): track 2.04 -> 0.00 mm
- net unconnected-(U2-PE10-PadB8): track 2.00 -> 0.00 mm
- net unconnected-(U2-PE9-PadB6): track 1.97 -> 0.00 mm
- net unconnected-(U2-PH14-PadB7): track 1.95 -> 0.00 mm
- net unconnected-(U2-PH9-PadA9): track 1.93 -> 0.00 mm
- net unconnected-(U2-PH13-PadA10): track 1.88 -> 0.00 mm
- net unconnected-(U2-PE7-PadA5): track 1.80 -> 0.00 mm
- net unconnected-(U1-PC11-PadB18): track 1.72 -> 0.00 mm
- net unconnected-(U2-PG4-PadA8): track 1.64 -> 0.00 mm
- net unconnected-(U2-PE8-PadA7): track 1.61 -> 0.00 mm
- net unconnected-(U2-PD5-PadA6): track 1.43 -> 0.00 mm
- net unconnected-(U1-PF0-PadA16): track 0.58 -> 0.00 mm, vias 1 -> 0
Other:
- copper layers 2 -> 6
- board text added: "26-pin Raspberry Pi Header"
- board text added: "Analog/Digital Placeholders"
- board text added: "CAN"
- board text added: "DC/DC Converters"
- board text added: "DDR3 DRAM x16"
- board text added: "MX34"
- board text added: "NAND Flash"
- board text added: "Power Input"
- board text added: "RS232"
- board text added: "RTC"
- board text added: "Soc"

Commit message: morning
Parts:
- added REF**: PQFP-256_28x28mm_P0.4mm, Package_QFP:PQFP-256_28x28mm_P0.4mm, F.Cu at (150.8, 95.8)

Commit message: pc night
Parts:
- removed REF**: PQFP-256_28x28mm_P0.4mm, Package_QFP:PQFP-256_28x28mm_P0.4mm
- added H1: MountingHole_Pad, MountingHole:MountingHole_3.2mm_M3_Pad, F.Cu at (176.1, 62.6)
- added H2: MountingHole_Pad, MountingHole:MountingHole_3.2mm_M3_Pad, F.Cu at (114.6, 124.0)
- added H3: MountingHole_Pad, MountingHole:MountingHole_3.2mm_M3_Pad, F.Cu at (114.2, 62.4)
- added H4: MountingHole_Pad, MountingHole:MountingHole_3.2mm_M3_Pad, F.Cu at (176.1, 123.9)
- C1, C2, C3, C4, C5, C6, R5: moved to B.Cu
- moved U1 105.3 mm to (59.6, 172.9)
- moved U2 105.3 mm to (76.1, 173.6)
- moved J3 101.3 mm to (120.7, 73.0), turned to 90 degrees
- moved J1 70.0 mm to (129.3, 80.9)
- moved C10 69.2 mm to (128.6, 70.9)
- moved C7 69.2 mm to (141.2, 65.4)
- moved C8 69.2 mm to (143.4, 65.4)
- moved C9 69.2 mm to (133.6, 61.5)
- moved D1 69.2 mm to (138.1, 61.7)
- moved L1 69.2 mm to (126.4, 64.2)
- moved R1 69.2 mm to (132.6, 68.6)
- moved R2 69.2 mm to (134.7, 68.6)
- moved U6 69.2 mm to (136.2, 65.3)
- moved U4 67.2 mm to (128.6, 122.9)
- moved C11 58.2 mm to (165.9, 65.2)
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Other:
- board outline added: 70 x 70 mm

Commit message: laptop morning
Parts:
- moved C9 78.8 mm to (137.0, 140.2), turned to -90 degrees
- moved D1 78.5 mm to (132.5, 140.0), turned to 0 degrees
- moved C13 78.1 mm to (160.2, 139.4), turned to -90 degrees
- moved D2 78.0 mm to (155.7, 139.2), turned to 0 degrees
- moved L1 74.9 mm to (142.8, 137.4), turned to 90 degrees
- moved L2 74.0 mm to (165.9, 136.5), turned to 90 degrees
- moved C8 72.8 mm to (127.1, 136.3), turned to 90 degrees
- moved C12 72.6 mm to (150.3, 135.5), turned to 90 degrees
- moved C7 71.9 mm to (129.4, 136.3), turned to 90 degrees
- moved C11 71.6 mm to (152.6, 135.5), turned to 90 degrees
- moved U6 71.3 mm to (134.3, 136.5), turned to 180 degrees
- moved U9 70.7 mm to (157.5, 135.6), turned to 180 degrees
- moved R1 64.5 mm to (136.5, 133.0), turned to 180 degrees
- moved R2 64.4 mm to (134.5, 133.0), turned to 180 degrees
- moved R3 63.8 mm to (159.7, 132.1), turned to 180 degrees
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Other:
- board size 70 x 70 mm -> 75 x 75 mm
- copper layers 6 -> 8
- board text added: "+3V3"
- board text added: "+5V"
- board text added: "DRAM"
- board text added: "FLASH"
- board text added: "POWER"
- board text added: "RPI"
- board text added: "SoC"
- board text added: "V_{IN}"
