File: spacex-sbc.kicad_pcb (KiCad board)
At the start: 8 copper layers, 75 x 75 mm, 44 parts, among them J1 26PIN_RPI_HEADER, J2 MX34 40-PIN, J3 Conn_01x02, U1 STM32MP135AAFx, U10 MCP16501TE-E/RMB, U11 MT40A512M16JY, U2 STM32MP131AAEx, U3 ATSAMA5D21, U4 MAX3221, U5 MT41K256M16TW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

Commit message: after rough draft submission
Parts:
- added REF**: BatteryHolder_Multicomp_BC-2001_1x2032, Battery:BatteryHolder_Multicomp_BC-2001_1x2032, B.Cu at (21.9, 187.9)
- added RTC BATTERY: BatteryHolder_LINX_BAT-HLD-012-SMT, Battery:BatteryHolder_LINX_BAT-HLD-012-SMT, F.Cu at (178.7, 113.9)
- Y1: footprint Crystal:Crystal_SMD_1210-4Pin_1.2x1.0mm -> Crystal:Crystal_SMD_2520-4Pin_2.5x2.0mm
- moved U10 6.35 mm to (172.3, 130.3)
- moved C11 4.17 mm to (148.5, 136.2)
- moved C12 4.17 mm to (146.2, 136.2)
- moved C16 4.17 mm to (159.7, 130.5)
- moved L2 4.17 mm to (161.8, 137.2)
- moved R3 4.17 mm to (155.6, 132.8)
- moved R4 4.17 mm to (153.6, 132.8)
- moved U9 4.17 mm to (153.4, 136.4)
- moved C13 4.17 mm to (156.1, 140.1)
- moved D2 4.17 mm to (151.6, 139.9)
- moved C7 3.25 mm to (126.1, 136.3)
- moved C9 3.25 mm to (133.7, 140.2)
- moved D1 3.25 mm to (129.2, 140.0)
- moved L1 3.25 mm to (139.5, 137.3)
- moved U6 3.25 mm to (131.0, 136.5)
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Connections:
- net DDR_CLK renamed DDR_CLKP
- J1 pad 1: Net-(J1-Pin_1) -> +3V3
- J1 pad 17: Net-(J1-Pin_1) -> +3V3
- U11 pad K7: unconnected-(U11-CK_t-PadK7) -> FLASH_WE
- U11 pad K8: unconnected-(U11-CK_c-PadK8) -> FLASH_PR
Routing:
- net GND: track 0.00 -> 20.0 mm
- net XIN: track 0.00 -> 6.49 mm
- net XOUT: track 0.00 -> 4.83 mm
- net unconnected-(U10-VI-Pad1): vias 0 -> 1
- net unconnected-(U10-GND-Pad2): vias 0 -> 1
- net (no net): vias 0 -> 77
