File: mx34.kicad_sch (KiCad schematic)
At the start: 1 part, among them J2 MX34 40-PIN

Commit message: before caleb
Connections:
- net CANH: now also J2.b4 (Pin_b4); no longer J2.a9 (Pin_a9)
- net CANL: now also J2.b5 (Pin_b5); no longer J2.a10 (Pin_a10)
- net RS232_DOUT: now also J2.a9 (Pin_a9); no longer J2.b4 (Pin_b4)
- net RS232_RIN: now also J2.a10 (Pin_a10); no longer J2.b5 (Pin_b5)
