File: ram.kicad_sch (KiCad schematic)
At the start: 2 parts, among them U5 MT41K256M16TW

Commit message: morning
Connections:
- no-connect marks 0 -> 1
Changed lines of the file:
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@@
 		(color 0 0 0 0)
+	)
+	(no_connect
+		(at 138.43 91.44)
 	)
 	(wire

Commit message: after rough draft submission
Connections:
- net DDR_CLK renamed DDR_CLKP
Changed lines of the file:
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@@
 		)
 	)
-	(global_label "DDR_CLK"
+	(global_label "DDR_CLKP"
 		(shape output)
 		(at 132.08 132.08 180)
