File: spacex-sbc.kicad_sch (KiCad schematic)
At the start: 1 part, among them J1 Conn_02x13_Odd_Even

Commit message: saved
Parts:
- added U1: STM32MP135AAFx, Package_BGA:ST_TFBGA-320_11x11mm_Layout21x21_P0.5mm, symbol MCU_ST_STM32MP1:STM32MP135AAFx
- added U2: ATSAMA5D21, Package_BGA:ST_LFBGA-354_16x16mm_Layout19x19_P0.8mm, symbol MCU_Microchip_SAMA:ATSAMA5D21
Connections:
- new net: U2.D7 (VDDIOP0), U2.F4 (VDDIOP0)
- new net: U2.E4 (GNDIOP0), U2.E7 (GNDIOP0)
- new net: U2.E8 (VDDCORE), U2.G8 (VDDCORE), U2.H8 (VDDCORE), U2.H9 (VDDCORE), U2.J5 (VDDCORE)
- new net: U2.F8 (GNDCORE), U2.G7 (GNDCORE), U2.G9 (GNDCORE), U2.H7 (GNDCORE), U2.J4 (GNDCORE)
- new net: U2.H2 (VDDANA), U2.K3 (VDDANA)
- new net: U2.J2 (GNDANA), U2.K4 (GNDANA)
- new net: U2.K8 (VDDIOP1), U2.L11 (VDDIOP1)
- new net: U2.K9 (GNDIOP1), U2.L12 (GNDIOP1)
- new net: U1.A1 (VSS), U1.A21 (VSS), U1.AA1 (VSS), U1.AA21 (VSS), U1.B12 (VSS), U1.D16 (VSS), U1.E11 (VSS), U1.E16 (VSS), U1.E5 (VSS), U1.E6 (VSS), U1.F17 (VSS), U1.F18 (VSS), U1.F21 (VSS), U1.F5 (VSS), U1.G12 (VSS), U1.G14 (VSS), U1.G8 (VSS), U1.H15 (VSS), U1.H7 (VSS), U1.J10 (VSS), U1.J12 (VSS), U1.K10 (VSS), U1.K11 (VSS), U1.K12 (VSS), U1.K13 (VSS), U1.K21 (VSS), U1.K9 (VSS), U1.L10 (VSS), U1.L12 (VSS), U1.L15 (VSS), U1.L17 (VSS), U1.L5 (VSS), U1.M1 (VSS), U1.M10 (VSS), U1.M11 (VSS), U1.M12 (VSS), U1.M13 (VSS), U1.M7 (VSS), U1.M9 (VSS), U1.N11 (VSS), U1.P15 (VSS), U1.P7 (VSS), U1.R11 (VSS), U1.R14 (VSS), U1.R8 (VSS), U1.T1 (VSS), U1.T17 (VSS), U1.T21 (VSS), U1.T5 (VSS), U1.U11 (VSS), U1.U13 (VSS), U1.U16 (VSS), U1.U5 (VSS), U1.U6 (VSS), U1.V16 (VSS), U1.W16 (VSS)
- new net: U2.C12 (DDR_VREF), U2.H12 (DDR_VREF)
- new net: U2.C6 (VDDIODDR), U2.E10 (VDDIODDR), U2.E12 (VDDIODDR), U2.G10 (VDDIODDR), U2.G12 (VDDIODDR), U2.H11 (VDDIODDR), U2.J10 (VDDIODDR)
- new net: U2.C7 (GNDIODDR), U2.D12 (GNDIODDR), U2.E9 (GNDIODDR), U2.F12 (GNDIODDR), U2.G11 (GNDIODDR), U2.H10 (GNDIODDR), U2.J11 (GNDIODDR)

Commit message: mostly mocked up
Parts:
- removed J1: Conn_02x13_Odd_Even, Connector_PinSocket_2.54mm:PinSocket_2x13_P2.54mm_Vertical, symbol Connector_Generic:Conn_02x13_Odd_Even
- removed U1: STM32MP135AAFx, Package_BGA:ST_TFBGA-320_11x11mm_Layout21x21_P0.5mm, symbol MCU_ST_STM32MP1:STM32MP135AAFx
- removed U2: ATSAMA5D21, Package_BGA:ST_LFBGA-354_16x16mm_Layout19x19_P0.8mm, symbol MCU_Microchip_SAMA:ATSAMA5D21
Other:
- added sheet Analog (analog.kicad_sch)
- added sheet CAN (can.kicad_sch)
- added sheet Digital (digital.kicad_sch)
- added sheet Flash (flash.kicad_sch)
- added sheet MX34 (mx34.kicad_sch)
- added sheet Pi Header (rpi.kicad_sch)
- added sheet Power (power.kicad_sch)
- added sheet RAM (ram.kicad_sch)
- added sheet RS232 (rs232.kicad_sch)
- added sheet RTC (rtc.kicad_sch)
- added sheet SoC (soc.kicad_sch)
- note added: "blank"
- company: (none) -> Austin Driggs
- title: (none) -> SpaceX SBC

Commit message: pc night
Parts:
- added H1, H2, H3, H4: MountingHole_Pad, MountingHole:MountingHole_3.2mm_M3_Pad, symbol Mechanical:MountingHole_Pad
Connections:
- new net GND: H1.1, H2.1, H3.1, H4.1
